Commit message: add dual arm benchmark, find collision bug

File: curobo/content/assets/robot/franka_description/dual_franka.urdf (robot description, URDF)
Before this commit: robot dual_franka, 31 links, 30 joints
Joints:
- joint world_to_left_arm: origin xyz=-0.4 0 0 rpy=0 0 0 -> xyz=0 -0.4 0 rpy=0 0 1.57079632679
- joint world_to_right_arm: origin xyz=0.4 0 0 rpy=0 0 3.14159265359 -> xyz=0 0.4 0 rpy=0 0 -1.57079632679
