Commit message: add dual arm relative pose cost and dual franka urdf with attached object collision spheres

File: curobo/content/assets/robot/franka_description/curobo_base_qhdu3yjn_dual_franka.urdf (robot description, URDF)
Before this commit: robot dual_franka, 33 links, 32 joints
Joints:
- joint world_to_left_arm: origin xyz=0 -0.4 0 rpy=0 0 1.57079632679 -> xyz=0.0 -0.444 0.0 rpy=0.0 0.0 1.5707771464270195
- joint world_to_right_arm: origin xyz=0 0.4 0 rpy=0 0 -1.57079632679 -> xyz=0.0 0.444 0.0 rpy=0.0 0.0 -1.5707771464270195
