Commit message: add wrist_camera and collision models

File: curobo/content/assets/robot/franka_description/dual_franka_with_camera.urdf (robot description, URDF)
Before this commit: robot dual_franka, 33 links, 32 joints
Links:
- added link panda_left_wrist_camera; visual mesh filename=meshes/visual/wrist_camera.STL
- added link panda_right_wrist_camera; visual mesh filename=meshes/visual/wrist_camera.STL
Joints:
- added joint panda_left_wrist_camera_joint: type fixed, parent panda_left_link8, child panda_left_wrist_camera, origin xyz=0 0 0 rpy=0 0 -0.785398163397, axis 0 0 0
- added joint panda_right_wrist_camera_joint: type fixed, parent panda_right_link8, child panda_right_wrist_camera, origin xyz=0 0 0 rpy=0 0 -0.785398163397, axis 0 0 0
- joint panda_left_hand_joint: origin xyz=0 0 0 rpy=0 0 -0.785398163397 -> xyz=0 0 0.003 rpy=0 0 0; parent panda_left_link8 -> panda_left_wrist_camera
- joint panda_right_hand_joint: origin xyz=0 0 0 rpy=0 0 -0.785398163397 -> xyz=0 0 0.003 rpy=0 0 0; parent panda_right_link8 -> panda_right_wrist_camera
- joint world_to_left_arm: origin xyz=0.0 -0.444 0.0 rpy=0.0 0.0 1.5707771464270195 -> xyz=0 -0.4 0 rpy=0 0 1.57079632679
- joint world_to_right_arm: origin xyz=0.0 0.444 0.0 rpy=0.0 0.0 -1.5707771464270195 -> xyz=0 -0.4 0 rpy=0 0 -1.57079632679
