Commit message: feat: dual-arm reactive MPC with coordinated motion
- Add dual_arm_viz.py: reactive MPC + Viser for dual-arm Panda
- Add Coordinate button: merge control frames for coordinated dual-arm motion
- Add gen_scene_1/2.py: parametric scene generators
- Add 5 scene configs (myscene_1~5.yml) and my_scene.yml
- Add dual_panda.yml, mj_left/right_arm.yml robot configs
- Add dual_franka_panda.urdf, mj_*_arm.urdf with camera meshes
- Fix dual_franka_with_camera.urdf right arm Y position
- Add run.md documentation
- Add test_dual_panda.py test script

Co-Authored-By: Claude <noreply@anthropic.com>

File: curobo/content/assets/robot/franka_description/dual_franka_panda.urdf (robot description, URDF)
Before this commit: robot dual_franka, 35 links, 34 joints
Links:
- removed link panda_left_base_link
- removed link panda_left_ee_link
- removed link panda_left_gripper
- removed link panda_left_hand
- removed link panda_left_hand_tcp
- removed link panda_left_leftfinger
- removed link panda_left_link0
- removed link panda_left_link1
- removed link panda_left_link2
- removed link panda_left_link3
- removed link panda_left_link4
- removed link panda_left_link5
- removed link panda_left_link6
- removed link panda_left_link7
- removed link panda_left_link8
- removed link panda_left_rightfinger
- removed link panda_left_wrist_camera
- removed link panda_right_base_link
- removed link panda_right_ee_link
- removed link panda_right_gripper
- removed link panda_right_hand
- removed link panda_right_hand_tcp
- removed link panda_right_leftfinger
- removed link panda_right_link0
- removed link panda_right_link1
- removed link panda_right_link2
- removed link panda_right_link3
- removed link panda_right_link4
- removed link panda_right_link5
- removed link panda_right_link6
- removed link panda_right_link7
- removed link panda_right_link8
- removed link panda_right_rightfinger
- removed link panda_right_wrist_camera
- removed link world_base_link
- added link left_ee_link
- added link left_panda_gripper, mass 0.01
- added link left_panda_hand, mass 1.0; collision mesh filename=meshes/collision/hand.obj; visual mesh filename=meshes/visual/hand.dae
- added link left_panda_leftfinger; collision mesh filename=meshes/collision/finger.obj; visual mesh filename=meshes/visual/finger.dae
- added link left_panda_link0, mass 2.3966; collision mesh filename=meshes/collision/link0.obj; visual mesh filename=meshes/visual/link0.dae
- added link left_panda_link1, mass 2.797; collision mesh filename=meshes/collision/link1.obj; visual mesh filename=meshes/visual/link1.dae
- added link left_panda_link2, mass 2.542; collision mesh filename=meshes/collision/link2.obj; visual mesh filename=meshes/visual/link2.dae
- added link left_panda_link3, mass 2.2513; collision mesh filename=meshes/collision/link3.obj; visual mesh filename=meshes/visual/link3.dae
- added link left_panda_link4, mass 2.2037; collision mesh filename=meshes/collision/link4.obj; visual mesh filename=meshes/visual/link4.dae
- added link left_panda_link5, mass 2.2855; collision mesh filename=meshes/collision/link5.obj; visual mesh filename=meshes/visual/link5.dae
- added link left_panda_link6, mass 1.353; collision mesh filename=meshes/collision/link6.obj; visual mesh filename=meshes/visual/link6.dae
- added link left_panda_link7, mass 0.35973; collision mesh filename=meshes/collision/link7.obj; visual mesh filename=meshes/visual/link7.dae
- added link left_panda_link8
- added link left_panda_rightfinger; collision mesh filename=meshes/collision/finger.obj; visual mesh filename=meshes/visual/finger.dae
- added link right_ee_link
- added link right_panda_gripper, mass 0.01
- added link right_panda_hand, mass 1.0; collision mesh filename=meshes/collision/hand.obj; visual mesh filename=meshes/visual/hand.dae
- added link right_panda_leftfinger; collision mesh filename=meshes/collision/finger.obj; visual mesh filename=meshes/visual/finger.dae
- added link right_panda_link0, mass 2.3966; collision mesh filename=meshes/collision/link0.obj; visual mesh filename=meshes/visual/link0.dae
- added link right_panda_link1, mass 2.797; collision mesh filename=meshes/collision/link1.obj; visual mesh filename=meshes/visual/link1.dae
- added link right_panda_link2, mass 2.542; collision mesh filename=meshes/collision/link2.obj; visual mesh filename=meshes/visual/link2.dae
- added link right_panda_link3, mass 2.2513; collision mesh filename=meshes/collision/link3.obj; visual mesh filename=meshes/visual/link3.dae
- added link right_panda_link4, mass 2.2037; collision mesh filename=meshes/collision/link4.obj; visual mesh filename=meshes/visual/link4.dae
- added link right_panda_link5, mass 2.2855; collision mesh filename=meshes/collision/link5.obj; visual mesh filename=meshes/visual/link5.dae
- added link right_panda_link6, mass 1.353; collision mesh filename=meshes/collision/link6.obj; visual mesh filename=meshes/visual/link6.dae
- added link right_panda_link7, mass 0.35973; collision mesh filename=meshes/collision/link7.obj; visual mesh filename=meshes/visual/link7.dae
- added link right_panda_link8
- added link right_panda_rightfinger; collision mesh filename=meshes/collision/finger.obj; visual mesh filename=meshes/visual/finger.dae
- added link world
Joints:
- removed joint panda_left_ee_fixed_joint
- removed joint panda_left_finger_joint1
- removed joint panda_left_finger_joint2
- removed joint panda_left_fixed
- removed joint panda_left_gripper_joint
- removed joint panda_left_hand_joint
- removed joint panda_left_hand_tcp_joint
- removed joint panda_left_joint1
- removed joint panda_left_joint2
- removed joint panda_left_joint3
- removed joint panda_left_joint4
- removed joint panda_left_joint5
- removed joint panda_left_joint6
- removed joint panda_left_joint7
- removed joint panda_left_joint8
- removed joint panda_left_wrist_camera_joint
- removed joint panda_right_ee_fixed_joint
- removed joint panda_right_finger_joint1
- removed joint panda_right_finger_joint2
- removed joint panda_right_fixed
- removed joint panda_right_gripper_joint
- removed joint panda_right_hand_joint
- removed joint panda_right_hand_tcp_joint
- removed joint panda_right_joint1
- removed joint panda_right_joint2
- removed joint panda_right_joint3
- removed joint panda_right_joint4
- removed joint panda_right_joint5
- removed joint panda_right_joint6
- removed joint panda_right_joint7
- removed joint panda_right_joint8
- removed joint panda_right_wrist_camera_joint
- removed joint world_to_left_arm
- removed joint world_to_right_arm
- added joint left_ee_fixed_joint: type fixed, parent left_panda_hand, child left_ee_link, origin xyz=0.0 0. 0.1 rpy=0 0.0 0
- added joint left_panda_finger_joint1: type prismatic, parent left_panda_hand, child left_panda_leftfinger, origin xyz=0 0 0.0584 rpy=0 0 0, axis 0 1 0, limit lower=0.0 upper=0.04 effort=20 velocity=0.2
- added joint left_panda_finger_joint2: type prismatic, parent left_panda_hand, child left_panda_rightfinger, origin xyz=0 0 0.0584 rpy=0 0 0, axis 0 -1 0, limit lower=0.0 upper=0.04 effort=20 velocity=0.2
- added joint left_panda_fixed: type fixed, parent world, child left_panda_link0, origin xyz=0 0.26 0 rpy=0 0 0.0, axis 0 0 0
- added joint left_panda_gripper_joint: type fixed, parent left_panda_link7, child left_right_gripper, origin xyz=0 0 0.207 rpy=0 0 2.35619449019, axis 0 0 1
- added joint left_panda_hand_joint: type fixed, parent left_panda_link8, child left_panda_hand, origin xyz=0 0 0 rpy=0 0 -0.785398163397
- added joint left_panda_joint1: type revolute, parent left_panda_link0, child left_panda_link1, origin xyz=0 0 0.333 rpy=0 0 0, axis 0 0 1, limit lower=-2.8973 upper=2.8973 effort=87 velocity=2.1750
- added joint left_panda_joint2: type revolute, parent left_panda_link1, child left_panda_link2, origin xyz=0 0 0 rpy=-1.57079632679 0 0, axis 0 0 1, limit lower=-1.7628 upper=1.7628 effort=87 velocity=2.1750
- added joint left_panda_joint3: type revolute, parent left_panda_link2, child left_panda_link3, origin xyz=0 -0.316 0 rpy=1.57079632679 0 0, axis 0 0 1, limit lower=-2.8973 upper=2.8973 effort=87 velocity=2.1750
- added joint left_panda_joint4: type revolute, parent left_panda_link3, child left_panda_link4, origin xyz=0.0825 0 0 rpy=1.57079632679 0 0, axis 0 0 1, limit lower=-3.0718 upper=-0.0698 effort=87 velocity=2.1750
- added joint left_panda_joint5: type revolute, parent left_panda_link4, child left_panda_link5, origin xyz=-0.0825 0.384 0 rpy=-1.57079632679 0 0, axis 0 0 1, limit lower=-2.8973 upper=2.8973 effort=12 velocity=2.6100
- added joint left_panda_joint6: type revolute, parent left_panda_link5, child left_panda_link6, origin xyz=0 0 0 rpy=1.57079632679 0 0, axis 0 0 1, limit lower=-0.0175 upper=3.7525 effort=12 velocity=2.6100
- added joint left_panda_joint7: type revolute, parent left_panda_link6, child left_panda_link7, origin xyz=0.088 0 0 rpy=1.57079632679 0 0, axis 0 0 1, limit lower=-2.8973 upper=2.8973 effort=12 velocity=2.6100
- added joint left_panda_joint8: type fixed, parent left_panda_link7, child left_panda_link8, origin xyz=0 0 0.107 rpy=0 0 0, axis 0 0 0
- added joint right_ee_fixed_joint: type fixed, parent right_panda_hand, child right_ee_link, origin xyz=0.0 0. 0.1 rpy=0 0.0 0
- added joint right_panda_finger_joint1: type prismatic, parent right_panda_hand, child right_panda_leftfinger, origin xyz=0 0 0.0584 rpy=0 0 0, axis 0 1 0, limit lower=0.0 upper=0.04 effort=20 velocity=0.2
- added joint right_panda_finger_joint2: type prismatic, parent right_panda_hand, child right_panda_rightfinger, origin xyz=0 0 0.0584 rpy=0 0 0, axis 0 -1 0, limit lower=0.0 upper=0.04 effort=20 velocity=0.2
- added joint right_panda_fixed: type fixed, parent world, child right_panda_link0, origin xyz=0 -0.26 0 rpy=0 0 0.0, axis 0 0 0
- added joint right_panda_gripper_joint: type fixed, parent right_panda_link7, child right_right_gripper, origin xyz=0 0 0.207 rpy=0 0 2.35619449019, axis 0 0 1
- added joint right_panda_hand_joint: type fixed, parent right_panda_link8, child right_panda_hand, origin xyz=0 0 0 rpy=0 0 -0.785398163397
- added joint right_panda_joint1: type revolute, parent right_panda_link0, child right_panda_link1, origin xyz=0 0 0.333 rpy=0 0 0, axis 0 0 1, limit lower=-2.8973 upper=2.8973 effort=87 velocity=2.1750
- added joint right_panda_joint2: type revolute, parent right_panda_link1, child right_panda_link2, origin xyz=0 0 0 rpy=-1.57079632679 0 0, axis 0 0 1, limit lower=-1.7628 upper=1.7628 effort=87 velocity=2.1750
- added joint right_panda_joint3: type revolute, parent right_panda_link2, child right_panda_link3, origin xyz=0 -0.316 0 rpy=1.57079632679 0 0, axis 0 0 1, limit lower=-2.8973 upper=2.8973 effort=87 velocity=2.1750
- added joint right_panda_joint4: type revolute, parent right_panda_link3, child right_panda_link4, origin xyz=0.0825 0 0 rpy=1.57079632679 0 0, axis 0 0 1, limit lower=-3.0718 upper=-0.0698 effort=87 velocity=2.1750
- added joint right_panda_joint5: type revolute, parent right_panda_link4, child right_panda_link5, origin xyz=-0.0825 0.384 0 rpy=-1.57079632679 0 0, axis 0 0 1, limit lower=-2.8973 upper=2.8973 effort=12 velocity=2.6100
- added joint right_panda_joint6: type revolute, parent right_panda_link5, child right_panda_link6, origin xyz=0 0 0 rpy=1.57079632679 0 0, axis 0 0 1, limit lower=-0.0175 upper=3.7525 effort=12 velocity=2.6100
- added joint right_panda_joint7: type revolute, parent right_panda_link6, child right_panda_link7, origin xyz=0.088 0 0 rpy=1.57079632679 0 0, axis 0 0 1, limit lower=-2.8973 upper=2.8973 effort=12 velocity=2.6100
- added joint right_panda_joint8: type fixed, parent right_panda_link7, child right_panda_link8, origin xyz=0 0 0.107 rpy=0 0 0, axis 0 0 0
